File: KiCad/Sally2/Sally2.kicad_sch (KiCad schematic)
At the start: 34 parts, among them J1 Power SW, J10 GND +5V, J11 A16, J2 Power LED, J3 USB_B, J4 PowerIn, J5 GND +5V, J6 Barrel_Jack, J7 GND +5V, J9 + A14 -, SW1 Reset, U1 GAL16V8 - IO decoder, U2 Z80ACPU, U3 GAL16V8 - ADR decoder, U4 27C256, U5 628128_DIP32_SSOP32, U6 GAL16V8 - glue logic, U7 74LS259, X1 16Mhz

Commit message: KiCad merges from Marc
Parts:
- removed J1: Power SW, Connector_PinHeader_2.54mm:PinHeader_1x02_P2.54mm_Vertical, symbol Connector_Generic:Conn_01x02
- removed J2: Power LED, Connector_PinHeader_2.54mm:PinHeader_1x02_P2.54mm_Vertical, symbol Connector_Generic:Conn_01x02
- added C14, C15, C16, C17, C18, C19, C20, C21, C22: ,1µ, Capacitor_THT:C_Disc_D5.0mm_W2.5mm_P5.00mm, symbol Device:C
- added J1: Conn_02x05_Odd_Even, Connector_PinHeader_2.54mm:PinHeader_2x05_P2.54mm_Horizontal, symbol Connector_Generic:Conn_02x05_Odd_Even
- added J21: - +, Sally2:BKL_1x2 72510U_P2.5mm_Vertical, symbol Connector_Generic:Conn_01x02
- added J22: A18, Connector_PinHeader_2.54mm:PinHeader_1x02_P2.54mm_Vertical, symbol AtariXL:Conn_01x02_Male
- added J23: CS2 / A17, Connector_PinHeader_2.54mm:PinHeader_1x02_P2.54mm_Vertical, symbol AtariXL:Conn_01x02_Male
- C2, C3, C4, C5, C6, C7, C8: value 100nF -> ,1µ
- J10, J5, J7: value GND +5V -> - +; footprint Connector_PinHeader_2.54mm:PinHeader_1x02_P2.54mm_Vertical -> Sally2:BKL_1x2 72510U_P2.5mm_Vertical
- J4: value PowerIn -> - +; footprint Connector_PinHeader_2.54mm:PinHeader_1x02_P2.54mm_Vertical -> Sally2:BKL_1x2 72510U_P2.5mm_Vertical
- U4: value 27C256 -> 27C128(256)
- U5: value 628128_DIP32_SSOP32 -> 62864(128/512)
- X1: footprint Package_DIP:DIP-14_W7.62mm -> Oscillator:Oscillator_DIP-14
Connections:
- net +5V: now also C14.1, C15.1, C16.1, C17.1, C18.1, C19.1, C20.1, C21.1, C22.1, J1.5 (Pin_5), J1.6 (Pin_6), J21.2 (Pin_2), J23.2 (Pin_2); no longer J5.2 (Pin_2), J7.2 (Pin_2), U5.30 (CS2)
- net GND: now also C14.2, C15.2, C16.2, C17.2, C18.2, C19.2, C20.2, C21.2, C22.2, J1.3 (Pin_3), J1.4 (Pin_4), J21.1 (Pin_1), J22.2 (Pin_2); no longer J3.4 (GND)
- net RES SW: now reaches R13.2, SW1.2
- net at J3.1 (VBUS), J6.1: now also J7.2 (Pin_2), J1.1 (Pin_1), J1.2 (Pin_2); no longer J4.2 (Pin_2)
- net at J6.3 (MountPin): now also J3.4 (GND)
- net at U5.1 (~{n.c.}): now also J22.1 (Pin_1)
- new net: J23.1 (Pin_1), U5.30 (CS2)
- new net: J1.10 (Pin_10), J1.9 (Pin_9), J5.2 (Pin_2)
- new net: J1.7 (Pin_7), J1.8 (Pin_8), J4.2 (Pin_2)
- no-connect marks 0 -> 14
Other:
- note added: "SALLY Prototyp 2"
- note removed: "ROM\ = MemRq + A15 + A14 + A13 + !RomEna + RD RAM0\ = MemRq + A15 + !(A14 + A13 + !RomEna + RD) RAM1\ = MemRq + !A15"
- moved on the sheet: C1, C2, C3, C4, C5, C6, C7, C8, J10, J4, J5, J7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
